File: hardware/quad.brd (EAGLE design)
At the start: 160 x 100 mm, 1 part, among them U101 STM32F427VGT6

Commit message: Continue work on schematic
Parts:
- added C1, C2: (no value), quad:C0603
- added C10, C5, C6, C7, C8, C9: 100nF, quad:C0603
- added C11, C12: 1uF, quad:C0603
- added C3, C4: 2.2uF, quad:C0603
- added R1: (no value), quad:R0603
- added U$1: PUSHBUTTON_SMD, quad:PUSHBUTTON_SMD
- added X101: 24MHz, quad:OSC3.2X2.5
Connections:
- removed net BOOT0: U101.94
- removed net NRST: U101.14
- removed net OSC_IN: U101.12
- removed net OSC_OUT: U101.13
- removed net VCAP2: U101.73
- removed net VCAP_1: U101.49
- removed net VDD: U101.100, U101.11, U101.19, U101.28, U101.50, U101.75
- removed net VDDA: U101.22
- removed net VREF+: U101.21
- removed net VSS: U101.10, U101.27, U101.74, U101.99
- removed net VSSA: U101.20
- new net GND: C1.1, C10.2, C11.2, C12.2, C2.2, C3.2, C4.2, C5.2, C6.2, C7.2, C8.2, C9.2, U$1.3, U$1.4, U101.10, U101.20, U101.27, U101.74, U101.94, U101.99, X101.2, X101.4
- new net N$1: C1.2, U101.12, X101.1
- new net N$2: C2.1, U101.13, X101.3
- new net N$3: R1.1, U$1.1, U$1.2, U101.14
- new net N$4: C3.1, U101.73
- new net N$5: C4.1, U101.49
- new net N$7: C11.1, U101.21
- new net VDD_3V3: C10.1, C12.1, C5.1, C6.1, C7.1, C8.1, C9.1, R1.2, U101.100, U101.11, U101.19, U101.22, U101.28, U101.50, U101.75
Changed lines of the file:
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@@
 <layer number="97" name="Info" color="7" fill="1" visible="no" active="no"/>
 <layer number="98" name="Guide" color="6" fill="1" visible="no" active="no"/>
+<layer number="99" name="SpiceOrder" color="5" fill="1" visible="no" active="no"/>
 </layers>
 <board>
@@
 <elements>
 <element name="U101" library="quad" package="LQFP-100" value="STM32F427VGT6" x="11.43" y="-10.16"/>
+<element name="X101" library="quad" package="OSC3.2X2.5" value="24MHz" x="8.89" y="-24.13"/>
+<element name="C1" library="quad" package="C0603" value="" x="3.81" y="-30.48"/>
+<element name="C2" library="quad" package="C0603" value="" x="3.81" y="-34.29"/>
+<element name="R1" library="quad" package="R0603" value="" x="2.54" y="-38.1"/>
+<element name="U$1" library="quad" package="PUSHBUTTON_SMD" value="PUSHBUTTON_SMD" x="6.35" y="-43.18"/>
+<element name="C3" library="quad" package="C0603" value="2.2uF" x="3.81" y="-49.53"/>
+<element name="C4" library="quad" package="C0603" value="2.2uF" x="3.81" y="-53.34"/>
+<element name="C5" library="quad" package="C0603" value="100nF" x="3.81" y="-57.15"/>
+<element name="C6" library="quad" package="C0603" value="100nF" x="3.81" y="-60.96"/>
+<element name="C7" library="quad" package="C0603" value="100nF" x="3.81" y="-64.77"/>
+<element name="C8" library="quad" package="C0603" value="100nF" x="3.81" y="-68.58"/>
+<element name="C9" library="quad" package="C0603" value="100nF" x="3.81" y="-72.39"/>
+<element name="C10" library="quad" package="C0603" value="100nF" x="3.81" y="-76.2"/>
+<element name="C11" library="quad" package="C0603" value="1uF" x="3.81" y="-80.01"/>
+<element name="C12" library="quad" package="C0603" value="1uF" x="3.81" y="-85.09"/>
 </elements>
 <signals>
@@
 <contactref element="U101" pad="46"/>
 </signal>
-<signal name="OSC_IN">
-<contactref element="U101" pad="12"/>
-</signal>
-<signal name="OSC_OUT">
-<contactref element="U101" pad="13"/>
-</signal>
-<signal name="NRST">
-<contactref element="U101" pad="14"/>
-</signal>
-<signal name="BOOT0">
+<signal name="VBAT">
+<contactref element="U101" pad="6"/>
+</signal>
+<signal name="OSC2">
+</signal>
+<signal name="OSC1">
+</signal>
+<signal name="GND">
+<contactref element="C2" pad="2"/>
+<contactref element="C1" pad="1"/>
+<contactref element="X101" pad="4"/>
+<contactref element="X101" pad="2"/>
 <contactref element="U101" pad="94"/>
-</signal>
-<signal name="VCAP_1">
-<contactref element="U101" pad="49"/>
-</signal>
-<signal name="VCAP2">
-<contactref element="U101" pad="73"/>
-</signal>
-<signal name="VSS">
-<contactref element="U101" pad="10"/>
-<contactref element="U101" pad="27"/>
+<contactref element="U$1" pad="4"/>
+<contactref element="U$1" pad="3"/>
+<contactref element="C3" pad="2"/>
+<contactref element="C4" pad="2"/>
 <contactref element="U101" pad="74"/>
 <contactref element="U101" pad="99"/>
-<wire x1="5.93" y1="-2.4384" x2="19.1516" y2="-4.66" width="0" layer="19" extent="1-1"/>
-<wire x1="3.7084" y1="-8.66" x2="5.93" y2="-2.4384" width="0" layer="19" extent="1-1"/>
-<wire x1="5.93" y1="-17.8816" x2="3.7084" y2="-8.66" width="0" layer="19" extent="1-1"/>
-</signal>
-<signal name="VDD">
-<contactref element="U101" pad="50"/>
-<contactref element="U101" pad="11"/>
-<contactref element="U101" pad="19"/>
-<contactref element="U101" pad="28"/>
+<contactref element="U101" pad="27"/>
+<contactref element="U101" pad="10"/>
+<contactref element="C5" pad="2"/>
+<contactref element="C6" pad="2"/>
+<contactref element="C7" pad="2"/>
+<contactref element="C8" pad="2"/>
+<contactref element="C9" pad="2"/>
+<contactref element="C10" pad="2"/>
+<contactref element="U101" pad="20"/>
+<contactref element="C11" pad="2"/>
+<contactref element="C12" pad="2"/>
+<wire x1="4.66" y1="-80.01" x2="4.66" y2="-85.09" width="0" layer="19" extent="1-1"/>
+<wire x1="4.66" y1="-76.2" x2="4.66" y2="-80.01" width="0" layer="19" extent="1-1"/>
+<wire x1="4.66" y1="-72.39" x2="4.66" y2="-76.2" width="0" layer="19" extent="1-1"/>
+<wire x1="4.66" y1="-68.58" x2="4.66" y2="-72.39" width="0" layer="19" extent="1-1"/>
+<wire x1="4.66" y1="-64.77" x2="4.66" y2="-68.58" width="0" layer="19" extent="1-1"/>
+<wire x1="4.66" y1="-60.96" x2="4.66" y2="-64.77" width="0" layer="19" extent="1-1"/>
+<wire x1="4.66" y1="-57.15" x2="4.66" y2="-60.96" width="0" layer="19" extent="1-1"/>
+<wire x1="4.66" y1="-53.34" x2="4.66" y2="-57.15" width="0" layer="19" extent="1-1"/>
+<wire x1="4.66" y1="-49.53" x2="4.66" y2="-53.34" width="0" layer="19" extent="1-1"/>
+<wire x1="3.25" y1="-45.03" x2="4.66" y2="-49.53" width="0" layer="19" extent="1-1"/>
+<wire x1="9.45" y1="-45.03" x2="3.25" y2="-45.03" width="0" layer="19" extent="1-1"/>
+<wire x1="4.66" y1="-34.29" x2="3.25" y2="-45.03" width="0" layer="19" extent="1-1"/>
+<wire x1="2.96" y1="-30.48" x2="4.66" y2="-34.29" width="0" layer="19" extent="1-1"/>
+<wire x1="6.096" y1="-22.098" x2="2.96" y2="-30.48" width="0" layer="19" extent="1-1"/>
+<wire x1="5.93" y1="-17.8816" x2="6.096" y2="-22.098" width="0" layer="19" extent="1-1"/>
+<wire x1="3.7084" y1="-13.66" x2="5.93" y2="-17.8816" width="0" layer="19" extent="1-1"/>
+<wire x1="3.7084" y1="-8.66" x2="3.7084" y2="-13.66" width="0" layer="19" extent="1-1"/>
+<wire x1="5.93" y1="-2.4384" x2="3.7084" y2="-8.66" width="0" layer="19" extent="1-1"/>
+<wire x1="8.43" y1="-2.4384" x2="5.93" y2="-2.4384" width="0" layer="19" extent="1-1"/>
+<wire x1="11.684" y1="-26.162" x2="6.096" y2="-22.098" width="0" layer="19" extent="1-1"/>
+<wire x1="19.1516" y1="-4.66" x2="8.43" y2="-2.4384" width="0" layer="19" extent="1-1"/>
+</signal>
+<signal name="N$1">
+<contactref element="U101" pad="12"/>
+<contactref element="X101" pad="1"/>
+<contactref element="C1" pad="2"/>
+<wire x1="6.096" y1="-26.162" x2="4.66" y2="-30.48" width="0" layer="19" extent="1-1"/>
+<wire x1="3.7084" y1="-9.66" x2="6.096" y2="-26.162" width="0" layer="19" extent="1-1"/>
+</signal>
+<signal name="N$2">
+<contactref element="X101" pad="3"/>
+<contactref element="U101" pad="13"/>
+<contactref element="C2" pad="1"/>
+<wire x1="11.684" y1="-22.098" x2="2.96" y2="-34.29" width="0" layer="19" extent="1-1"/>
+<wire x1="3.7084" y1="-10.16" x2="11.684" y2="-22.098" width="0" layer="19" extent="1-1"/>
+</signal>
+<signal name="N$3">
+<contactref element="U101" pad="14"/>
+<contactref element="R1" pad="1"/>
+<contactref element="U$1" pad="2"/>
+<contactref element="U$1" pad="1"/>
+<wire x1="3.25" y1="-41.33" x2="1.69" y2="-38.1" width="0" layer="19" extent="1-1"/>
+<wire x1="9.45" y1="-41.33" x2="3.25" y2="-41.33" width="0" layer="19" extent="1-1"/>
+<wire x1="3.7084" y1="-10.66" x2="1.69" y2="-38.1" width="0" layer="19" extent="1-1"/>
+</signal>
+<signal name="VDD_3V3">
+<contactref element="R1" pad="2"/>
 <contactref element="U101" pad="75"/>
 <contactref element="U101" pad="100"/>
-<wire x1="5.43" y1="-2.4384" x2="19.1516" y2="-4.16" width="0" layer="19" extent="1-1"/>
-<wire x1="3.7084" y1="-9.16" x2="5.43" y2="-2.4384" width="0" layer="19" extent="1-1"/>
-<wire x1="3.7084" y1="-13.16" x2="3.7084" y2="-9.16" width="0" layer="19" extent="1-1"/>
-<wire x1="6.43" y1="-17.8816" x2="3.7084" y2="-13.16" width="0" layer="19" extent="1-1"/>
+<contactref element="U101" pad="19"/>
+<contactref element="U101" pad="11"/>
+<contactref element="U101" pad="28"/>
+<contactref element="U101" pad="50"/>
+<contactref element="C10" pad="1"/>
+<contactref element="C9" pad="1"/>
+<contactref element="C8" pad="1"/>
+<contactref element="C7" pad="1"/>
+<contactref element="C6" pad="1"/>
+<contactref element="C5" pad="1"/>
+<contactref element="U101" pad="22"/>
+<contactref element="C12" pad="1"/>
+<wire x1="2.96" y1="-76.2" x2="2.96" y2="-85.09" width="0" layer="19" extent="1-1"/>
+<wire x1="2.96" y1="-72.39" x2="2.96" y2="-76.2" width="0" layer="19" extent="1-1"/>
+<wire x1="2.96" y1="-68.58" x2="2.96" y2="-72.39" width="0" layer="19" extent="1-1"/>
+<wire x1="2.96" y1="-64.77" x2="2.96" y2="-68.58" width="0" layer="19" extent="1-1"/>
+<wire x1="2.96" y1="-60.96" x2="2.96" y2="-64.77" width="0" layer="19" extent="1-1"/>
+<wire x1="2.96" y1="-57.15" x2="2.96" y2="-60.96" width="0" layer="19" extent="1-1"/>
+<wire x1="3.39" y1="-38.1" x2="2.96" y2="-57.15" width="0" layer="19" extent="1-1"/>
+<wire x1="6.43" y1="-17.8816" x2="3.39" y2="-38.1" width="0" layer="19" extent="1-1"/>
+<wire x1="3.7084" y1="-14.66" x2="6.43" y2="-17.8816" width="0" layer="19" extent="1-1"/>
+<wire x1="3.7084" y1="-13.16" x2="3.7084" y2="-14.66" width="0" layer="19" extent="1-1"/>
+<wire x1="3.7084" y1="-9.16" x2="3.7084" y2="-13.16" width="0" layer="19" extent="1-1"/>
+<wire x1="5.43" y1="-2.4384" x2="3.7084" y2="-9.16" width="0" layer="19" extent="1-1"/>
 <wire x1="17.43" y1="-17.8816" x2="6.43" y2="-17.8816" width="0" layer="19" extent="1-1"/>
-</signal>
-<signal name="VDDA">
-<contactref element="U101" pad="22"/>
-</signal>
-<signal name="VREF+">
+<wire x1="19.1516" y1="-4.16" x2="5.43" y2="-2.4384" width="0" layer="19" extent="1-1"/>
+</signal>
+<signal name="N$4">
+<contactref element="U101" pad="73"/>
+<contactref element="C3" pad="1"/>
+<wire x1="19.1516" y1="-5.16" x2="2.96" y2="-49.53" width="0" layer="19" extent="1-1"/>
+</signal>
+<signal name="N$5">
+<contactref element="U101" pad="49"/>
+<contactref element="C4" pad="1"/>
+<wire x1="16.93" y1="-17.8816" x2="2.96" y2="-53.34" width="0" layer="19" extent="1-1"/>
+</signal>
+<signal name="N$7">
+<contactref element="C11" pad="1"/>
 <contactref element="U101" pad="21"/>
-</signal>
-<signal name="VSSA">
-<contactref element="U101" pad="20"/>
-</signal>
-<signal name="VBAT">
-<contactref element="U101" pad="6"/>
+<wire x1="3.7084" y1="-14.16" x2="2.96" y2="-80.01" width="0" layer="19" extent="1-1"/>
 </signal>
 </signals>
