File: hardware/quad.brd (EAGLE design)
At the start: 254 x 254 mm, 68 parts, among them IC1 BNO055, J501 I2C_TEST, U101 STM32F427VGT6, U202 AND_GATE, U203 SN74AHC1G32DBVR, U401 FT232R, U402 USB-MICROB, U403 LD1117, U404 MFS201N-16-Z, X101 24MHz, Y501 32.768kHz

Commit message: Redo board power layout
Parts:
- removed BNO_NBOOTLD, BNO_NRST: TESTPAD, quad:TESTPAD
- moved C203 4.94 mm to (20.9, -2.24), turned to 0 degrees
- moved C210 4.51 mm to (8.13, -32.0), turned to 180 degrees
- moved C502 4.08 mm to (-8.26, 3.10), turned to 270 degrees
- moved U202 3.45 mm to (-2.16, -28.8), turned to 225 degrees
- moved U203 3.08 mm to (-7.16, -15.4), turned to 270 degrees
- moved C206 2.58 mm to (1.24, -19.7), turned to 135 degrees
- moved R201 2.44 mm to (0.23, -32.5), turned to 315 degrees
- moved C209 2.32 mm to (26.8, -15.3), turned to 90 degrees
- moved C205 2.07 mm to (-1.02, -11.2), turned to 90 degrees
- moved R101 1.88 mm to (22.4, -22.7), turned to 45 degrees
- moved R701 1.79 mm to (-42.2, 27.2), turned to 315 degrees
- moved C202 1.76 mm to (11.4, -29.4), turned to 0 degrees
- moved C211 1.57 mm to (28.8, -7.47), turned to 180 degrees
- moved C207 1.22 mm to (16.0, -2.26)
- moved C208 0.88 mm to (17.3, -26.3)
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- renumbered U$1 to J701, U$2 to U701
Connections:
- removed net N$13: BNO_NRST.P$1, IC1.11
- net N$16: no longer BNO_NBOOTLD.P$1
- net VBATT: now also U404.1; no longer U404.3
- net VBUS: now also U404.3; no longer U404.1
- net XBEE_DIO4: now also U404.4; no longer U404.6
Routing:
- net VDD_3V3: track 342.2 -> 483.2 mm, vias 4 -> 5
- net FT232_RTS: track 114.4 -> 89.7 mm
- net KILL_GND: track 274.4 -> 253.7 mm, vias 1 -> 2
- net USART1_TX: track 74.8 -> 54.7 mm
- net XBEE_DIO4: track 112.0 -> 92.3 mm, vias 1 -> 2
- net USART1_RX: track 82.5 -> 63.6 mm
- net USART3_TX: track 61.8 -> 73.0 mm
- net USART3_RX: track 65.3 -> 76.5 mm
- net VBATT: track 252.3 -> 260.8 mm, vias 0 -> 1
- net TIM3_CH1: track 93.5 -> 85.5 mm
- net FT232_DTR: track 99.8 -> 92.2 mm
- net TIM3_CH3: track 40.7 -> 46.9 mm, vias 0 -> 1
- net N$16: track 14.0 -> 8.84 mm
- net N$13: track 4.41 -> 0.00 mm
- net XBEE_DIO0: track 43.3 -> 45.2 mm, vias 0 -> 1
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- removed copper zone on layer 1, net VDD_3V3
