File: hardware/quad.brd (EAGLE design)
At the start: 254 x 254 mm, 66 parts, among them IC1 BNO055, J501 I2C_TEST, J701 XT60, U101 STM32F427VGT6, U202 AND_GATE, U203 SN74AHC1G32DBVR, U401 FT232R, U402 USB-MICROB, U403 LD1117, U404 MFS201N-16-Z, U701 PSMN9RS-30YLC, X101 24MHz, Y501 32.768kHz

Commit message: Minor changes
Parts:
- removed R5: 270, quad:R0603
- added JP1: (no value), quad:1X02
- added R404: 270, quad:R0603
- moved PWR 1.15 mm to (56.6, 18.3)
- moved EN 0.49 mm to (53.1, 14.5)
- renumbered RXLED to RX, TXLED to TX
Connections:
- net GND: now also R404.1; no longer R5.1
- net N$18: now also R404.2; no longer R5.2
- net USART1_RX: now also JP1.1
- net USART1_TX: now also JP1.2
Routing:
- net FT232_RTS: track 89.7 -> 93.3 mm
- net FT232_DTR: track 92.2 -> 95.7 mm
- net N$16: track 8.84 -> 5.92 mm
- net VDD_3V3: track 483.2 -> 480.6 mm, vias 5 -> 3
- net TIM3_CH4: track 65.6 -> 64.8 mm
- net N$18: track 1.75 -> 2.28 mm
- net N$19: track 2.74 -> 3.27 mm
- net USART1_RX: track 63.6 -> 63.4 mm, vias 2 -> 1
- net USART1_TX: vias 2 -> 1
- net GND: vias 62 -> 81
Other:
- board text added: "SCL"
- board text added: "SDA"
