File: hardware/quad.sch (EAGLE design)
At the start: 1 part, among them U101 STM32F427VGT6

Commit message: Continue work on schematic
Parts:
- added C1, C2: (no value), quad:C-EUC0603
- added C10, C5, C6, C7, C8, C9: 100nF, quad:C-EUC0603
- added C11, C12: 1uF, quad:C-EUC0603
- added C3, C4: 2.2uF, quad:C-EUC0603
- added R1: (no value), quad:R-US_R0603
- added U$1: PUSHBUTTON_SMD, quad:PUSHBUTTON_SMD
- added X101: 24MHz, quad:OSCILLATOR
Connections:
- new net GND: C1.1, C10.2, C11.2, C12.2, C2.2, C3.2, C4.2, C5.2, C6.2, C7.2, C8.2, C9.2, U$1.2, U101BATT.VSSA, U101RST.BOOT0, U101VCAP.VSS, X101.GND
- new net N$1: C1.2, U101OSC.OSC_IN, X101.OSC1
- new net N$2: C2.1, U101OSC.OSC_OUT, X101.OSC2
- new net N$3: R1.1, U$1.1, U101RST.NRST
- new net N$4: C3.1, U101VCAP.VCAP2
- new net N$5: C4.1, U101VCAP.VCAP_1
- new net N$7: C11.1, U101BATT.VREF+
- new net VDD_3V3: C10.1, C12.1, C5.1, C6.1, C7.1, C8.1, C9.1, R1.2, U101BATT.VDDA, U101VCAP.VDD
Other:
- note added: "Decoupling Capacitors Place as close to VDD pins as possible"
- note added: "STM32F4 IO Ports"
- note added: "STM32F4 Reset and Power"
