File: hardware/quad.sch (EAGLE design)
At the start: 66 parts, among them IC1 BNO055, J501 I2C_TEST, J701 XT60, U101 STM32F427VGT6, U202 AND_GATE, U203 SN74AHC1G32DBVR, U401 FT232R, U402 USB-MICROB, U403 LD1117, U404 MFS201N-16-Z, U701 PSMN9RS-30YLC, X101 24MHz, Y501 32.768kHz

Commit message: Minor changes
Parts:
- added JP1: (no value), quad:PINHD-1X2
- renumbered R5 to R404, RXLED to RX, TXLED to TX
Connections:
- net USART1_RX: now also JP1.1
- net USART1_TX: now also JP1.2
Other:
- moved on the sheet: U202, U203
